File: hardware/de0-orpsoc.brd (EAGLE design)
At the start: 75.2 x 49 mm, 101 parts, among them J1 J0026, J2 J0026, U1 USD-SOCKETNEW, U10 DS1307SO8, U2 MIC280, U3 KSZ8081RNA, U4 KSZ8851SNL, U5 USB1T11A, U7 TPS2552, Y1 32.768k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

Commit message: hw: fix osc cap value
Parts:
- C13, C14, C16, C31: value 18p -> 33p
- C17, C18: value 22p -> 33p
Changed lines of the file:
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@@
 <variant name="no-eth" populate="no"/>
 </element>
-<element name="C17" library="rcl" package="C0603" value="22p" x="51.0032" y="39.0144" rot="R270">
+<element name="C17" library="rcl" package="C0603" value="33p" x="51.0032" y="39.0144" rot="R270">
 <variant name="no-eth" populate="no"/>
 </element>
-<element name="C18" library="rcl" package="C0603" value="22p" x="43.4848" y="39.0144" rot="R90">
+<element name="C18" library="rcl" package="C0603" value="33p" x="43.4848" y="39.0144" rot="R90">
 <variant name="no-eth" populate="no"/>
 </element>
@@
 <element name="C11" library="rcl" package="C0603" value=".1u" x="51.6128" y="9.144" rot="R270"/>
 <element name="C12" library="rcl" package="C0603" value=".1u" x="43.2816" y="13.6144" rot="MR270"/>
-<element name="C16" library="rcl" package="C0603" value="18p" x="52.2224" y="20.7264" rot="R270"/>
-<element name="C31" library="rcl" package="C0603" value="18p" x="44.9072" y="20.7264" rot="R90"/>
+<element name="C16" library="rcl" package="C0603" value="33p" x="52.2224" y="20.7264" rot="R270"/>
+<element name="C31" library="rcl" package="C0603" value="33p" x="44.9072" y="20.7264" rot="R90"/>
 <element name="LED5" library="led" package="CHIPLED_0805" value="" x="67.2592" y="3.8608" rot="R180"/>
 <element name="R6" library="rcl" package="R0603" value="330" x="49.3776" y="10.3632" rot="MR180"/>
@@
 <element name="U$5" library="SparkFun-DigitalIC" package="LQFP-48" value="FT2232D" x="17.4752" y="34.1376" rot="R270"/>
 <element name="Y4" library="SparkFun" package="CRYSTAL-SMD-5X3" value="6MHz" x="16.8656" y="41.4528"/>
-<element name="C13" library="rcl" package="C0603" value="18p" x="13.208" y="41.4528" rot="R90"/>
-<element name="C14" library="rcl" package="C0603" value="18p" x="20.7264" y="41.4528" rot="R270"/>
+<element name="C13" library="rcl" package="C0603" value="33p" x="13.208" y="41.4528" rot="R90"/>
+<element name="C14" library="rcl" package="C0603" value="33p" x="20.7264" y="41.4528" rot="R270"/>
 <element name="C28" library="rcl" package="C0603" value="100n" x="18.0848" y="33.9344" rot="MR270">
 <variant name="no-eth" populate="no"/>

Commit message: hw: misc value fixes
Parts:
- C19: value 10u -> 100n
- Y3: value 25M -> 25MHz
Changed lines of the file:
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@@
 <variant name="no-eth" populate="no"/>
 </element>
-<element name="Y3" library="SparkFun" package="CRYSTAL-SMD-5X3" value="25M" x="47.3456" y="39.0144" rot="R180">
+<element name="Y3" library="SparkFun" package="CRYSTAL-SMD-5X3" value="25MHz" x="47.3456" y="39.0144" rot="R180">
 <variant name="no-eth" populate="no"/>
 </element>
@@
 <variant name="no-eth" populate="no"/>
 </element>
-<element name="C19" library="rcl" package="C0603" value="10u" x="54.864" y="37.7952" rot="R180">
+<element name="C19" library="rcl" package="C0603" value="100n" x="54.864" y="37.7952" rot="R180">
 <variant name="no-eth" populate="no"/>
 </element>

Commit message: hw: part values tweaks
Parts:
- C13, C14: value 33p -> dnp
- R30: value 22k -> 56k
- R31: value 15k -> 4k7
- R32: value 15k -> 10k
- R7, R8: value 27 -> 22
- U10: value DS1307SO8 -> DS1339
Changed lines of the file:
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@@
 <element name="R11" library="rcl" package="R0603" value="330" x="8.3312" y="2.4384" rot="R180"/>
 <element name="R12" library="rcl" package="R0603" value="330" x="8.3312" y="3.8608" rot="R180"/>
-<element name="U10" library="SparkFun-FreqCtrl" package="SO08" value="DS1307SO8" x="25.6032" y="18.6944" rot="R90"/>
+<element name="U10" library="SparkFun-FreqCtrl" package="SO08" value="DS1339" x="25.6032" y="18.6944" rot="R90"/>
 <element name="C3" library="rcl" package="C0603" value=".1u" x="23.9776" y="15.4432"/>
 <element name="Y1" library="SparkFun-FreqCtrl" package="CRYSTAL-32KHZ-SMD" value="32.768k" x="31.0896" y="17.4752" rot="R270"/>
@@
 <element name="U$5" library="SparkFun-DigitalIC" package="LQFP-48" value="FT2232D" x="17.4752" y="34.1376" rot="R270"/>
 <element name="Y4" library="SparkFun" package="CRYSTAL-SMD-5X3" value="6MHz" x="16.8656" y="41.4528"/>
-<element name="C13" library="rcl" package="C0603" value="33p" x="13.208" y="41.4528" rot="R90"/>
-<element name="C14" library="rcl" package="C0603" value="33p" x="20.7264" y="41.4528" rot="R270"/>
+<element name="C13" library="rcl" package="C0603" value="dnp" x="13.208" y="41.4528" rot="R90"/>
+<element name="C14" library="rcl" package="C0603" value="dnp" x="20.7264" y="41.4528" rot="R270"/>
 <element name="C28" library="rcl" package="C0603" value="100n" x="18.0848" y="33.9344" rot="MR270">
 <variant name="no-eth" populate="no"/>
@@
 <variant name="no-eth" populate="no"/>
 </element>
-<element name="R7" library="rcl" package="R0603" value="27" x="10.16" y="34.3408"/>
-<element name="R8" library="rcl" package="R0603" value="27" x="10.16" y="32.9184"/>
+<element name="R7" library="rcl" package="R0603" value="22" x="10.16" y="34.3408"/>
+<element name="R8" library="rcl" package="R0603" value="22" x="10.16" y="32.9184"/>
 <element name="R13" library="rcl" package="R0603" value="1k5" x="10.5664" y="35.7632" rot="R180"/>
 <element name="R14" library="rcl" package="R0603" value="5k6" x="10.5664" y="37.1856"/>
@@
 <element name="JP6" library="SparkFun-Connectors" package="USB-MICROB" value="USB_MICROB_PLUG" x="1.3716" y="26.8224" rot="R270"/>
 <element name="U7" library="balto" package="SOT23-6L" value="TPS2552" x="17.8816" y="24.384" rot="R90"/>
-<element name="R30" library="rcl" package="R0603" value="22k" x="14.224" y="24.1808" rot="R90"/>
-<element name="R31" library="rcl" package="R0603" value="15k" x="6.096" y="24.384" rot="R180"/>
-<element name="R32" library="rcl" package="R0603" value="15k" x="6.096" y="22.9616"/>
+<element name="R30" library="rcl" package="R0603" value="56k" x="14.224" y="24.1808" rot="R90"/>
+<element name="R31" library="rcl" package="R0603" value="4k7" x="6.096" y="24.384" rot="R180"/>
+<element name="R32" library="rcl" package="R0603" value="10k" x="6.096" y="22.9616"/>
 <element name="U$1" library="cat" package="CAT-L" value="" x="40.64" y="8.9408"/>
 <element name="U$4" library="cat" package="CS" value="" x="22.1488" y="24.384"/>

Commit message: hw: change rtc pn
Parts:
- U10: value DS1339 -> M41T82
Changed lines of the file:
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@@
 <element name="R11" library="rcl" package="R0603" value="330" x="8.3312" y="2.4384" rot="R180"/>
 <element name="R12" library="rcl" package="R0603" value="330" x="8.3312" y="3.8608" rot="R180"/>
-<element name="U10" library="SparkFun-FreqCtrl" package="SO08" value="DS1339" x="25.6032" y="18.6944" rot="R90"/>
+<element name="U10" library="SparkFun-FreqCtrl" package="SO08" value="M41T82" x="25.6032" y="18.6944" rot="R90"/>
 <element name="C3" library="rcl" package="C0603" value=".1u" x="23.9776" y="15.4432"/>
 <element name="Y1" library="SparkFun-FreqCtrl" package="CRYSTAL-32KHZ-SMD" value="32.768k" x="31.0896" y="17.4752" rot="R270"/>
