File: hardware/de0-orpsoc.sch (EAGLE design)
At the start: 99 parts, among them J1 J0026, J2 J0026, U1 USD-SOCKETNEW, U10 DS1307SO8, U2 MIC280, U3 KSZ8081RNA, U4 KSZ8851SNL, U5 USB1T11A, U7 TPS2552, Y1 32.768k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

Commit message: hw: fix osc cap value
Parts:
- C13, C14, C16, C31: value 18p -> 33p
- C17, C18: value 22p -> 33p
Changed lines of the file:
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@@
 <variant name="no-eth" populate="no"/>
 </part>
-<part name="C17" library="rcl" deviceset="C-EU" device="C0603" value="22p">
+<part name="C17" library="rcl" deviceset="C-EU" device="C0603" value="33p">
 <variant name="no-eth" populate="no"/>
 </part>
-<part name="C18" library="rcl" deviceset="C-EU" device="C0603" value="22p">
+<part name="C18" library="rcl" deviceset="C-EU" device="C0603" value="33p">
 <variant name="no-eth" populate="no"/>
 </part>
@@
 <part name="C12" library="rcl" deviceset="C-EU" device="C0603" value=".1u"/>
 <part name="GND23" library="supply1" deviceset="GND" device=""/>
-<part name="C16" library="rcl" deviceset="C-EU" device="C0603" value="18p"/>
-<part name="C31" library="rcl" deviceset="C-EU" device="C0603" value="18p"/>
+<part name="C16" library="rcl" deviceset="C-EU" device="C0603" value="33p"/>
+<part name="C31" library="rcl" deviceset="C-EU" device="C0603" value="33p"/>
 <part name="LED5" library="led" deviceset="LED" device="CHIPLED_0805"/>
 <part name="R6" library="rcl" deviceset="R-EU_" device="R0603" value="330"/>
@@
 <part name="GND26" library="supply1" deviceset="GND" device=""/>
 <part name="GND27" library="supply1" deviceset="GND" device=""/>
-<part name="C13" library="rcl" deviceset="C-EU" device="C0603" value="18p"/>
-<part name="C14" library="rcl" deviceset="C-EU" device="C0603" value="18p"/>
+<part name="C13" library="rcl" deviceset="C-EU" device="C0603" value="33p"/>
+<part name="C14" library="rcl" deviceset="C-EU" device="C0603" value="33p"/>
 <part name="+3V17" library="supply1" deviceset="+3V3" device=""/>
 <part name="+3V18" library="supply1" deviceset="+3V3" device=""/>
@@
 <segment>
 <pinref part="JP5" gate="G$1" pin="1"/>
-<wire x1="241.3" y1="246.38" x2="228.6" y2="246.38" width="0.1524" layer="91"/>
-<label x="228.6" y="246.38" size="1.778" layer="95"/>
-</segment>
-<segment>
+<wire x1="241.3" y1="246.38" x2="223.52" y2="246.38" width="0.1524" layer="91"/>
+<label x="223.52" y="246.38" size="1.778" layer="95"/>
+</segment>
+<segment>

Commit message: hw: mark a yellow LED
Other:
- note added: "Green . . . . . ."
- note added: "Yellow"
- moved on the sheet: C2, C6, TP1, TP2, U2

Commit message: hw: misc value fixes
Parts:
- C19: value 10u -> 100n
- Y3: value 25M -> 25MHz
Changed lines of the file:
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@@
 <variant name="no-eth" populate="no"/>
 </part>
-<part name="Y3" library="SparkFun" deviceset="CRYSTAL" device="5X3" value="25M">
+<part name="Y3" library="SparkFun" deviceset="CRYSTAL" device="5X3" value="25MHz">
 <variant name="no-eth" populate="no"/>
 </part>
@@
 <variant name="no-eth" populate="no"/>
 </part>
-<part name="C19" library="rcl" deviceset="C-EU" device="C0603" value="10u">
+<part name="C19" library="rcl" deviceset="C-EU" device="C0603" value="100n">
 <variant name="no-eth" populate="no"/>
 </part>

Commit message: hw: part values tweaks
Parts:
- C13, C14: value 33p -> dnp
- R30: value 22k -> 56k
- R31: value 15k -> 4k7
- R32: value 15k -> 10k
- R7, R8: value 27 -> 22
- U10: value DS1307SO8 -> DS1339
Other:
- note added: "Green"
- note added: "Red"
- note removed: "732-3819-1-ND"
- note removed: "A106671-ND"
- note removed: "BK-890-ND 3mm 300-8340-1-ND"
- note removed: "EVQ-PLHA15"
- note removed: "Green . . . . . ."
- note removed: "USB1T11AM‑ND"
- note removed: "Yellow"
Changed lines of the file:
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@@
 <part name="R11" library="rcl" deviceset="R-EU_" device="R0603" value="330"/>
 <part name="R12" library="rcl" deviceset="R-EU_" device="R0603" value="330"/>
-<part name="U10" library="SparkFun-FreqCtrl" deviceset="DS1307" device="SO8"/>
+<part name="U10" library="SparkFun-FreqCtrl" deviceset="DS1307" device="SO8" value="DS1339"/>
 <part name="C3" library="rcl" deviceset="C-EU" device="C0603" value=".1u"/>
 <part name="GND6" library="supply1" deviceset="GND" device=""/>
@@
 <part name="GND26" library="supply1" deviceset="GND" device=""/>
 <part name="GND27" library="supply1" deviceset="GND" device=""/>
-<part name="C13" library="rcl" deviceset="C-EU" device="C0603" value="33p"/>
-<part name="C14" library="rcl" deviceset="C-EU" device="C0603" value="33p"/>
+<part name="C13" library="rcl" deviceset="C-EU" device="C0603" value="dnp"/>
+<part name="C14" library="rcl" deviceset="C-EU" device="C0603" value="dnp"/>
 <part name="+3V17" library="supply1" deviceset="+3V3" device=""/>
 <part name="+3V18" library="supply1" deviceset="+3V3" device=""/>
@@
 </part>
 <part name="GND28" library="supply1" deviceset="GND" device=""/>
-<part name="R7" library="rcl" deviceset="R-EU_" device="R0603" value="27"/>
-<part name="R8" library="rcl" deviceset="R-EU_" device="R0603" value="27"/>
+<part name="R7" library="rcl" deviceset="R-EU_" device="R0603" value="22"/>
+<part name="R8" library="rcl" deviceset="R-EU_" device="R0603" value="22"/>
 <part name="R13" library="rcl" deviceset="R-EU_" device="R0603" value="1k5"/>
 <part name="R14" library="rcl" deviceset="R-EU_" device="R0603" value="5k6"/>
@@
 <part name="GND50" library="supply1" deviceset="GND" device=""/>
 <part name="U7" library="balto" deviceset="TPS2552" device=""/>
-<part name="R30" library="rcl" deviceset="R-EU_" device="R0603" value="22k"/>
+<part name="R30" library="rcl" deviceset="R-EU_" device="R0603" value="56k"/>
 <part name="GND51" library="supply1" deviceset="GND" device=""/>
 <part name="GND52" library="supply1" deviceset="GND" device=""/>
 <part name="P+9" library="supply1" deviceset="+5V" device=""/>
-<part name="R31" library="rcl" deviceset="R-EU_" device="R0603" value="15k"/>
-<part name="R32" library="rcl" deviceset="R-EU_" device="R0603" value="15k"/>
+<part name="R31" library="rcl" deviceset="R-EU_" device="R0603" value="4k7"/>
+<part name="R32" library="rcl" deviceset="R-EU_" device="R0603" value="10k"/>
 <part name="GND53" library="supply1" deviceset="GND" device=""/>
 <part name="GND54" library="supply1" deviceset="GND" device=""/>
@@
 <wire x1="284.48" y1="139.7" x2="284.48" y2="88.9" width="0.1524" layer="97"/>
 <text x="287.02" y="132.08" size="5.08" layer="97">uSD</text>
-<text x="340.36" y="106.68" size="1.778" layer="97" rot="R90">732-3819-1-ND</text>
-<text x="170.18" y="195.58" size="1.778" layer="97">USB1T11AM‑ND</text>
 <text x="149.86" y="254" size="5.08" layer="97">USB</text>
 <wire x1="320.04" y1="261.62" x2="386.08" y2="261.62" width="0.1524" layer="97"/>
@@
 <wire x1="345.44" y1="142.24" x2="345.44" y2="88.9" width="0.1524" layer="97"/>
 <wire x1="345.44" y1="88.9" x2="386.08" y2="88.9" width="0.1524" layer="97"/>
-<text x="45.72" y="96.52" size="1.778" layer="97">BK-890-ND 3mm
-300-8340-1-ND</text>
-<text x="287.02" y="175.26" size="1.778" layer="97">EVQ-PLHA15</text>
-<text x="325.12" y="193.04" size="1.778" layer="97">A106671-ND</text>
-<text x="294.64" y="68.58" size="1.778" layer="97">Yellow</text>
+<text x="294.64" y="60.96" size="1.778" layer="97">Red</text>
 <text x="294.64" y="45.72" size="1.778" layer="97">Green
-.
-.
-.
-.
-.
-.</text>
+</text>
+<text x="294.64" y="68.58" size="1.778" layer="97">Green</text>
 </plain>
 <instances>

Commit message: hw: change rtc pn
Parts:
- U10: value DS1339 -> M41T82
Changed lines of the file:
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@@
 <part name="R11" library="rcl" deviceset="R-EU_" device="R0603" value="330"/>
 <part name="R12" library="rcl" deviceset="R-EU_" device="R0603" value="330"/>
-<part name="U10" library="SparkFun-FreqCtrl" deviceset="DS1307" device="SO8" value="DS1339"/>
+<part name="U10" library="SparkFun-FreqCtrl" deviceset="DS1307" device="SO8" value="M41T82"/>
 <part name="C3" library="rcl" deviceset="C-EU" device="C0603" value=".1u"/>
 <part name="GND6" library="supply1" deviceset="GND" device=""/>
